Commit message: Add rpy to all joints

File: hardware/URDF/robots/reachy.URDF (robot description, URDF)
Before this commit: robot Reachy, 9 links, 8 joints
Joints:
- joint arm_yaw: origin xyz=0 0 0 -> xyz=0 0 0 rpy=0 0 0
- joint ball_joint: origin xyz=0 0 -0.02409 -> xyz=0 0 -0.02409 rpy=0 0 0
- joint elbow_pitch: origin xyz=0 -0.0001 -0.30745 -> xyz=0 0 -0.30745 rpy=0 0 0
- joint forearm_yaw: origin xyz=0 0 0 -> xyz=0 0 0 rpy=0 0 0
- joint shoulder_pitch: origin xyz=0.0887 0 0 -> xyz=0.0887 0 0 rpy=0 0 0
- joint shoulder_roll: origin xyz=0 0 0 -> xyz=0 0 0 rpy=0 0 0
- joint wrist_pitch: origin xyz=0 0 -0.22415 -> xyz=0 0 -0.22415 rpy=0 0 0
- joint wrist_roll: origin xyz=0 0 -0.03243 -> xyz=0 0 -0.03243 rpy=0 0 0

Commit message: added axis to shoulder_pitch removed ball_joint joint not handled by ikpy

File: hardware/URDF/robots/reachy.URDF (robot description, URDF)
Before this commit: robot Reachy, 9 links, 8 joints
Joints:
- removed joint ball_joint
- joint shoulder_pitch: axis (none) -> 0 0 1

Commit message: axis corrected for shoulder_pitch added limit to all joints

File: hardware/URDF/robots/reachy.URDF (robot description, URDF)
Before this commit: robot Reachy, 9 links, 7 joints
Joints:
- joint arm_yaw: limit (none) -> lower=-1.5708 upper=1.5708
- joint elbow_pitch: limit (none) -> lower=0 upper=2.18166
- joint forearm_yaw: limit (none) -> lower=-2.61799 upper=2.61799
- joint shoulder_pitch: axis 0 0 1 -> 1 0 0; limit (none) -> lower=-1.5708 upper=3.14159
- joint shoulder_roll: limit (none) -> lower=-3.14159 upper=0.174533
- joint wrist_pitch: limit (none) -> lower=-1.22173 upper=1.22173
- joint wrist_roll: limit (none) -> lower=-1.0472 upper=1.0472

Commit message: modification of the URDF to fit the axis convention

File: hardware/URDF/robots/reachy.URDF (robot description, URDF)
Before this commit: robot Reachy, 9 links, 7 joints
Joints:
- joint arm_yaw: axis 0 0 -1 -> 0 0 1
- joint elbow_pitch: axis 1 0 0 -> 0 1 0; limit lower=0 upper=2.18166 -> lower=-2.18166 upper=0
- joint forearm_yaw: axis 0 0 -1 -> 0 0 1
- joint shoulder_pitch: axis 1 0 0 -> 0 1 0; origin xyz=0.0887 0 0 rpy=0 0 0 -> xyz=0 -0.0887 0 rpy=0 0 0
- joint shoulder_roll: axis 0 1 0 -> 1 0 0
- joint wrist_pitch: axis 1 0 0 -> 0 1 0
- joint wrist_roll: axis 0 1 0 -> 1 0 0

Commit message: update URDF with 3D models

File: hardware/URDF/robots/reachy.URDF (robot description, URDF)
Before this commit: robot Reachy, 9 links, 7 joints
Links:
- removed link ball
- link base: mass None -> 0.221; geometry collision mesh filename=package://meshes/shoulder-y-respondable.STL; visual mesh filename=package://meshes/shoulder-y-visual.STL
- link forearm: mass None -> 0.129; geometry collision mesh filename=package://meshes/forearm-respondable.STL; visual mesh filename=package://meshes/forearm-visual.STL
- link hand_ball: mass None -> 0.090; geometry collision mesh filename=package://meshes/ball-tip-respondable.STL; visual mesh filename=package://meshes/ball-tip-visual.STL
- link shoulder: mass None -> 0.036; geometry collision mesh filename=package://meshes/shoulder-respondable.STL; visual mesh filename=package://meshes/shoulder-visual.STL
- link shoulder_to_arm: mass None -> 0.155; geometry collision mesh filename=package://meshes/shoulder-x-respondable.STL; visual mesh filename=package://meshes/shoulder-x-visual.STL
- link upper_arm: mass None -> 0.430; geometry collision mesh filename=package://meshes/upper-arm-respondable.STL; visual mesh filename=package://meshes/upper-arm-visual.STL
- link wrist: mass None -> 0.115; geometry collision mesh filename=package://meshes/wrist-respondable.STL; visual mesh filename=package://meshes/wrist-visual.STL
- link wrist_hand: mass None -> 0.009; geometry collision mesh filename=package://meshes/wrist-hand-respondable.STL; visual mesh filename=package://meshes/wrist-hand-visual.STL
Joints:
- joint shoulder_pitch: origin xyz=0 -0.0887 0 rpy=0 0 0 -> xyz=0 -0.04 0 rpy=0 0 0
- joint wrist_pitch: origin xyz=0 0 -0.22415 rpy=0 0 0 -> xyz=0 0 -0.22425 rpy=0 0 0
