Commit message: update leachy URDF with 3D shapes

File: hardware/URDF/robots/leachy.URDF (robot description, URDF)
Before this commit: robot Reachy, 9 links, 7 joints
Links:
- removed link ball
- link base: mass None -> 0.221; geometry collision mesh filename=package://meshes/shoulder-y-left-respondable.STL; visual mesh filename=package://meshes/shoulder-y-left-visual.STL
- link forearm: mass None -> 0.129; geometry collision mesh filename=package://meshes/forearm-respondable.STL; visual mesh filename=package://meshes/forearm-visual.STL
- link hand_ball: mass None -> 0.090; geometry collision mesh filename=package://meshes/ball-tip-respondable.STL; visual mesh filename=package://meshes/ball-tip-visual.STL
- link shoulder: mass None -> 0.036; geometry collision mesh filename=package://meshes/shoulder-left-respondable.STL; visual mesh filename=package://meshes/shoulder-left-visual.STL
- link shoulder_to_arm: mass None -> 0.155; geometry collision mesh filename=package://meshes/shoulder-x-respondable.STL; visual mesh filename=package://meshes/shoulder-x-visual.STL
- link upper_arm: mass None -> 0.430; geometry collision mesh filename=package://meshes/upper-arm-respondable.STL; visual mesh filename=package://meshes/upper-arm-visual.STL
- link wrist: mass None -> 0.115; geometry collision mesh filename=package://meshes/wrist-respondable.STL; visual mesh filename=package://meshes/wrist-visual.STL
- link wrist_hand: mass None -> 0.009; geometry collision mesh filename=package://meshes/wrist-hand-respondable.STL; visual mesh filename=package://meshes/wrist-hand-visual.STL
