Commit message: Use new motor name with specific r_ or l_ prefix.

File: software/reachy/leachy.urdf (robot description, URDF)
Before this commit: robot Reachy, 8 links, 7 joints
Joints:
- removed joint arm_yaw
- removed joint elbow_pitch
- removed joint forearm_yaw
- removed joint shoulder_pitch
- removed joint shoulder_roll
- removed joint wrist_pitch
- removed joint wrist_roll
- added joint l_arm_yaw: type revolute, parent shoulder_to_arm, child upper_arm, origin xyz=0 0 0 rpy=0 0 0, axis 0 0 1, limit lower=-1.5708 upper=1.5708
- added joint l_elbow_pitch: type revolute, parent upper_arm, child forearm, origin xyz=0 0 -0.30745 rpy=0 0 0, axis 0 1 0, limit lower=-2.18166 upper=0
- added joint l_forearm_yaw: type revolute, parent forearm, child wrist, origin xyz=0 0 0 rpy=0 0 0, axis 0 0 1, limit lower=-2.61799 upper=2.61799
- added joint l_shoulder_pitch: type revolute, parent base, child shoulder, origin xyz=0 0.0887 0 rpy=0 0 0, axis 0 1 0, limit lower=-1.5708 upper=3.14159
- added joint l_shoulder_roll: type revolute, parent shoulder, child shoulder_to_arm, origin xyz=0 0 0 rpy=0 0 0, axis 1 0 0, limit lower=-0.174533 upper=3.14159
- added joint l_wrist_pitch: type revolute, parent wrist, child wrist_hand, origin xyz=0 0 -0.22415 rpy=0 0 0, axis 0 1 0, limit lower=-1.22173 upper=1.22173
- added joint l_wrist_roll: type revolute, parent wrist_hand, child hand_ball, origin xyz=0 0 -0.03243 rpy=0 0 0, axis 1 0 0, limit lower=-1.0472 upper=1.0472

File: software/reachy/reachy.urdf (robot description, URDF)
Before this commit: robot Reachy, 8 links, 7 joints
Joints:
- removed joint arm_yaw
- removed joint elbow_pitch
- removed joint forearm_yaw
- removed joint shoulder_pitch
- removed joint shoulder_roll
- removed joint wrist_pitch
- removed joint wrist_roll
- added joint r_arm_yaw: type revolute, parent shoulder_to_arm, child upper_arm, origin xyz=0 0 0 rpy=0 0 0, axis 0 0 1, limit lower=-1.5708 upper=1.5708
- added joint r_elbow_pitch: type revolute, parent upper_arm, child forearm, origin xyz=0 0 -0.30745 rpy=0 0 0, axis 0 1 0, limit lower=-2.18166 upper=0
- added joint r_forearm_yaw: type revolute, parent forearm, child wrist, origin xyz=0 0 0 rpy=0 0 0, axis 0 0 1, limit lower=-2.61799 upper=2.61799
- added joint r_shoulder_pitch: type revolute, parent base, child shoulder, origin xyz=0 -0.04 0 rpy=0 0 0, axis 0 1 0, limit lower=-1.5708 upper=3.14159
- added joint r_shoulder_roll: type revolute, parent shoulder, child shoulder_to_arm, origin xyz=0 0 0 rpy=0 0 0, axis 1 0 0, limit lower=-3.14159 upper=0.174533
- added joint r_wrist_pitch: type revolute, parent wrist, child wrist_hand, origin xyz=0 0 -0.22425 rpy=0 0 0, axis 0 1 0, limit lower=-1.22173 upper=1.22173
- added joint r_wrist_roll: type revolute, parent wrist_hand, child hand_ball, origin xyz=0 0 -0.03243 rpy=0 0 0, axis 1 0 0, limit lower=-1.0472 upper=1.0472

Commit message: Fix urdf file.

File: software/reachy/leachy.urdf (robot description, URDF)
Before this commit: robot Reachy, 8 links, 7 joints
Joints:
- joint l_shoulder_pitch: origin xyz=0 0.0887 0 rpy=0 0 0 -> xyz=0 0.14 0 rpy=0 0 0

File: software/reachy/leachy_hand.urdf (robot description, URDF)
Before this commit: robot Leachy w hand, 7 links, 6 joints
Joints:
- joint l_shoulder_pitch: origin xyz=0 0.0887 0 rpy=0 0 0 -> xyz=0 0.14 0 rpy=0 0 0

File: software/reachy/reachy_hand.urdf (robot description, URDF)
Before this commit: robot Reachy, 8 links, 7 joints
Links:
- removed link hand_ball
- removed link wrist_hand
- added link hand, mass 0.350; collision mesh filename=package://meshes/ball-tip-respondable.STL; visual mesh filename=package://meshes/ball-tip-visual.STL
Joints:
- removed joint r_wrist_roll
- joint r_wrist_pitch: child wrist_hand -> hand
